Commit message: updated to robot arm with ft sensor

File: trajopt_examples/assets/xarm6/xarm6_with_gripper.urdf (robot description, URDF)
Before this commit: robot xarm6_with_gripper, 17 links, 16 joints
Links:
- added link link_ft_sensor, mass 0.54156; collision mesh filename=file:///home/janne/phd1/xarm/src/xarm/xarm_ros/xarm_descrip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; visual mesh filename=file:///home/janne/phd1/xarm/src/xarm/xarm_ros/xarm_descrip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
Joints:
- added joint joint_ft_sensor: type fixed, parent link6, child link_ft_sensor, origin xyz=0 0 0.052 rpy=0 0 0
- joint joint_eef: parent link6 -> link_ft_sensor
